Commit message: Isaac ROS 4.0

File: isaac_ros_cumotion_examples/ur_config/ur.ros2_control.xacro (robot description, xacro)
@@ -10,6 +10,6 @@
       <joint name="${tf_prefix}shoulder_pan_joint">
         <command_interface name="position">
-          <param name="min">{-2*pi}</param>
-          <param name="max">{2*pi}</param>
+          <param name="min">-6.283185307179586</param>
+          <param name="max">6.283185307179586</param>
         </command_interface>
         <command_interface name="velocity">
@@ -25,6 +25,6 @@
       <joint name="${tf_prefix}shoulder_lift_joint">
         <command_interface name="position">
-          <param name="min">{-2*pi}</param>
-          <param name="max">{2*pi}</param>
+          <param name="min">-6.283185307179586</param>
+          <param name="max">6.283185307179586</param>
         </command_interface>
         <command_interface name="velocity">
@@ -55,6 +55,6 @@
       <joint name="${tf_prefix}wrist_1_joint">
         <command_interface name="position">
-          <param name="min">{-2*pi}</param>
-          <param name="max">{2*pi}</param>
+          <param name="min">-6.283185307179586</param>
+          <param name="max">6.283185307179586</param>
         </command_interface>
         <command_interface name="velocity">
@@ -70,6 +70,6 @@
       <joint name="${tf_prefix}wrist_2_joint">
         <command_interface name="position">
-          <param name="min">{-2*pi}</param>
-          <param name="max">{2*pi}</param>
+          <param name="min">-6.283185307179586</param>
+          <param name="max">6.283185307179586</param>
         </command_interface>
         <command_interface name="velocity">
@@ -85,6 +85,6 @@
       <joint name="${tf_prefix}wrist_3_joint">
         <command_interface name="position">
-          <param name="min">{-2*pi}</param>
-          <param name="max">{2*pi}</param>
+          <param name="min">-6.283185307179586</param>
+          <param name="max">6.283185307179586</param>
         </command_interface>
         <command_interface name="velocity">

File: isaac_ros_cumotion_robot_description/urdf/ur10e_robotiq_2f_140.urdf (robot description, URDF)
Before this commit: robot ur10e_robot, 24 links, 23 joints
Links:
- added link insertion_frame, mass 0.01
Joints:
- added joint insertion_joint: type fixed, parent gripper_frame, child insertion_frame, origin xyz=0 0 0.22 rpy=0 3.14 0

File: isaac_ros_cumotion_robot_description/urdf/ur10e_robotiq_2f_85.urdf (robot description, URDF)
Before this commit: robot robotiq_gripper, 25 links, 24 joints
Links:
- removed link ft_frame
- removed link world
- link base_link_inertia: geometry collision mesh filename=meshes/ur10e/collision/base.stl; visual mesh filename=meshes/ur10e/visual/base.dae
- link forearm_link: mass 2.275 -> 3.87; geometry collision mesh filename=meshes/ur10e/collision/forearm.stl; visual mesh filename=meshes/ur10e/visual/forearm.dae
- link shoulder_link: mass 3.7 -> 7.778; geometry collision mesh filename=meshes/ur10e/collision/shoulder.stl; visual mesh filename=meshes/ur10e/visual/shoulder.dae
- link upper_arm_link: mass 8.393 -> 12.93; geometry collision mesh filename=meshes/ur10e/collision/upperarm.stl; visual mesh filename=meshes/ur10e/visual/upperarm.dae
- link wrist_1_link: mass 1.219 -> 1.96; geometry collision mesh filename=meshes/ur10e/collision/wrist1.stl; visual mesh filename=meshes/ur10e/visual/wrist1.dae
- link wrist_2_link: mass 1.219 -> 1.96; geometry collision mesh filename=meshes/ur10e/collision/wrist2.stl; visual mesh filename=meshes/ur10e/visual/wrist2.dae
- link wrist_3_link: mass 0.1879 -> 0.202; geometry collision mesh filename=meshes/ur10e/collision/wrist3.stl; visual mesh filename=meshes/ur10e/visual/wrist3.dae
Joints:
- removed joint base_joint
- removed joint wrist_3_link-ft_frame
- joint elbow_joint: origin xyz=-0.425 0 0 rpy=0 0 0 -> xyz=-0.6127 0 0 rpy=0 0 0
- joint insertion_joint: origin xyz=0 0 0.22 rpy=0 3.14 0 -> xyz=0 0 0.15 rpy=0 3.14 0
- joint shoulder_lift_joint: limit lower=-6.283185307179586 upper=6.283185307179586 effort=150.0 velocity=3.141592653589793 -> lower=-6.283185307179586 upper=6.283185307179586 effort=330.0 velocity=2.0943951023931953
- joint shoulder_pan_joint: limit lower=-6.283185307179586 upper=6.283185307179586 effort=150.0 velocity=3.141592653589793 -> lower=-6.283185307179586 upper=6.283185307179586 effort=330.0 velocity=2.0943951023931953; origin xyz=0 0 0.1625 rpy=0 0 0 -> xyz=0 0 0.1807 rpy=0 0 0
- joint wrist_1_joint: limit lower=-6.283185307179586 upper=6.283185307179586 effort=28.0 velocity=3.141592653589793 -> lower=-6.283185307179586 upper=6.283185307179586 effort=56.0 velocity=3.141592653589793; origin xyz=-0.3922 0 0.1333 rpy=0 0 0 -> xyz=-0.57155 0 0.17415 rpy=0 0 0
- joint wrist_2_joint: limit lower=-6.283185307179586 upper=6.283185307179586 effort=28.0 velocity=3.141592653589793 -> lower=-6.283185307179586 upper=6.283185307179586 effort=56.0 velocity=3.141592653589793; origin xyz=0 -0.0997 -2.044881182297852e-11 rpy=1.570796327 0 0 -> xyz=0 -0.11985 -2.458164590756244e-11 rpy=1.570796327 0 0
- joint wrist_3_joint: limit lower=-6.283185307179586 upper=6.283185307179586 effort=28.0 velocity=3.141592653589793 -> lower=-6.283185307179586 upper=6.283185307179586 effort=56.0 velocity=3.141592653589793; origin xyz=0 0.0996 -2.042830148012698e-11 rpy=1.570796326589793 3.141592653589793 3.141592653589793 -> xyz=0 0.11655 -2.390480459346185e-11 rpy=1.570796326589793 3.141592653589793 3.141592653589793

File: isaac_ros_cumotion_robot_description/urdf/ur5e_robotiq_2f_140.urdf (robot description, URDF)
Before this commit: robot ur5e_robot, 24 links, 23 joints
Links:
- added link insertion_frame, mass 0.01
Joints:
- added joint insertion_joint: type fixed, parent gripper_frame, child insertion_frame, origin xyz=0 0 0.22 rpy=0 3.14 0
